Commit message: new urdf

File: spotmicroai.urdf (robot description, URDF)
Before this commit: robot differential_drive_robot, 23 links, 22 joints
Links:
- link base_link: geometry collision box size=0.14 0.11 0.07; visual mesh filename=/home/nico/aea_spot_micro/spot_micro/install/mobile_robot/s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 scale=0.001 0.001 0.001
- link front_left_foot_link: geometry collision box size=0.026 0.020 0.115; visual mesh filename=/home/nico/aea_spot_micro/spot_micro/install/mobile_robot/s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 scale=0.001 0.001 0.001
- link front_left_leg_link: geometry collision box size=0.028 0.036 0.12; visual mesh filename=/home/nico/aea_spot_micro/spot_micro/install/mobile_robot/s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 scale=0.001 0.001 0.001
- link front_left_leg_link_cover: geometry visual mesh filename=/home/nico/aea_spot_micro/spot_micro/install/mobile_robot/s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 scale=0.001 0.001 0.001
- link front_left_shoulder_link: geometry collision box size=0.044 0.038 0.07; visual mesh filename=/home/nico/aea_spot_micro/spot_micro/install/mobile_robot/s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 scale=0.001 0.001 0.001
- link front_left_toe_link: geometry collision sphere radius=0.02; visual mesh filename=/home/nico/aea_spot_micro/spot_micro/install/mobile_robot/s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 scale=0.001 0.001 0.001
- link front_link: geometry collision box size=0.058 0.11 0.07; visual mesh filename=/home/nico/aea_spot_micro/spot_micro/install/mobile_robot/s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 scale=0.001 0.001 0.001
- link front_right_foot_link: geometry collision box size=0.026 0.020 0.115; visual mesh filename=/home/nico/aea_spot_micro/spot_micro/install/mobile_robot/s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 scale=0.001 0.001 0.001
- link front_right_leg_link: geometry collision box size=0.028 0.036 0.12; visual mesh filename=/home/nico/aea_spot_micro/spot_micro/install/mobile_robot/s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 scale=0.001 0.001 0.001
- link front_right_leg_link_cover: geometry visual mesh filename=/home/nico/aea_spot_micro/spot_micro/install/mobile_robot/s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 scale=0.001 0.001 0.001
- link front_right_shoulder_link: geometry collision box size=0.044 0.038 0.07; visual mesh filename=/home/nico/aea_spot_micro/spot_micro/install/mobile_robot/s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 scale=0.001 0.001 0.001
- link front_right_toe_link: geometry collision sphere radius=0.02; visual mesh filename=/home/nico/aea_spot_micro/spot_micro/install/mobile_robot/s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 scale=0.001 0.001 0.001
- link rear_left_foot_link: geometry collision box size=0.026 0.020 0.115; visual mesh filename=/home/nico/aea_spot_micro/spot_micro/install/mobile_robot/s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 scale=0.001 0.001 0.001
- link rear_left_leg_link: geometry collision box size=0.028 0.036 0.12; visual mesh filename=/home/nico/aea_spot_micro/spot_micro/install/mobile_robot/s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 scale=0.001 0.001 0.001
- link rear_left_leg_link_cover: geometry visual mesh filename=/home/nico/aea_spot_micro/spot_micro/install/mobile_robot/s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 scale=0.001 0.001 0.001
- link rear_left_shoulder_link: geometry collision box size=0.044 0.038 0.07; visual mesh filename=/home/nico/aea_spot_micro/spot_micro/install/mobile_robot/s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 scale=0.001 0.001 0.001
- link rear_left_toe_link: geometry collision sphere radius=0.02; visual mesh filename=/home/nico/aea_spot_micro/spot_micro/install/mobile_robot/s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 scale=0.001 0.001 0.001
- link rear_link: geometry collision box size=0.04 0.11 0.07; visual mesh filename=/home/nico/aea_spot_micro/spot_micro/install/mobile_robot/s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 scale=0.001 0.001 0.001
- link rear_right_foot_link: geometry collision box size=0.026 0.020 0.115; visual mesh filename=/home/nico/aea_spot_micro/spot_micro/install/mobile_robot/s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 scale=0.001 0.001 0.001
- link rear_right_leg_link: geometry collision box size=0.028 0.036 0.12; visual mesh filename=/home/nico/aea_spot_micro/spot_micro/install/mobile_robot/s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 scale=0.001 0.001 0.001
- link rear_right_leg_link_cover: geometry visual mesh filename=/home/nico/aea_spot_micro/spot_micro/install/mobile_robot/s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 scale=0.001 0.001 0.001
- link rear_right_shoulder_link: geometry collision box size=0.044 0.038 0.07; visual mesh filename=/home/nico/aea_spot_micro/spot_micro/install/mobile_robot/s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 scale=0.001 0.001 0.001
- link rear_right_toe_link: geometry collision sphere radius=0.02; visual mesh filename=/home/nico/aea_spot_micro/spot_micro/install/mobile_robot/s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 scale=0.001 0.001 0.001
